Commit message: fix: Adapt URDF model to Planar Move Plugin
See http://gazebosim.org/tutorials?tut=ros_gzplugins.

File: topological_swarm/urdf/agent.xacro (robot description, xacro)
@@ -5,15 +5,29 @@
     <color rgba="1.0 1.0 1.0 1.0"/>
   </material>
-  <link name='base'>
-     <inertial>
-      <mass value="15.0"/>
-      <origin xyz="0.0 0 0" rpy=" 0 0 0"/>
-      <inertia
-          ixx="0.1" ixy="0" ixz="0"
-          iyy="0.1" iyz="0"
-          izz="0.1"
-      />
+  <!-- root link, on the ground just below the model origin -->
+  <link name="base_footprint">
+   <visual>
+      <origin xyz="0 0 0" rpy="0 0 0" />
+      <geometry>
+        <box size="0.01 0.01 0.01" />
+      </geometry>
+    </visual>
+    <material name="white"/>
+  </link>
+  <joint name="base_link_joint" type="fixed">
+    <origin xyz="0.0 0.0 0.0" rpy="0 0 0" />
+    <parent link="base_footprint"/>
+    <child link="base_link" />
+  </joint>
+  <!-- the spherical model -->
+  <link name="base_link">
+    <inertial>
+      <mass value="50" />
+      <origin xyz="0 0 0" />
+      <inertia ixx="50.0" ixy="0.0" ixz="0.0"
+        iyy="50.0" iyz="0.0"
+        izz="50.0" />
     </inertial>
-    <collision name='base_collision'>
+    <collision>
       <origin xyz="0 0 0" rpy=" 0 0 0"/>
       <geometry>
@@ -21,5 +35,5 @@
       </geometry>
     </collision>
-    <visual name='base_visual'>
+    <visual>
       <origin xyz="0 0 0" rpy=" 0 0 0"/>
       <geometry>

Commit message: feat: Add contact sensor to robot

File: topological_swarm/urdf/agent.xacro (robot description, xacro)
@@ -29,5 +29,5 @@
         izz="50.0" />
     </inertial>
-    <collision>
+    <collision name="base_link_collision">
       <origin xyz="0 0 0" rpy=" 0 0 0"/>
       <geometry>

Commit message: fix: Correct indentation

File: topological_swarm/urdf/agent.xacro (robot description, xacro)
@@ -7,5 +7,5 @@
   <!-- root link, on the ground just below the model origin -->
   <link name="base_footprint">
-   <visual>
+    <visual>
       <origin xyz="0 0 0" rpy="0 0 0" />
       <geometry>

Commit message: fix: Improve naming of collision elements
Change the names of collision elements in URDF and SDF so that
contact messages are generated correctly.

File: topological_swarm/urdf/agent.xacro (robot description, xacro)
@@ -29,5 +29,5 @@
         izz="50.0" />
     </inertial>
-    <collision name="base_link_collision">
+    <collision>
       <origin xyz="0 0 0" rpy=" 0 0 0"/>
       <geometry>
